File: doc/schematic/LED_Advent_wreath_deco/LED_Advent_wreath_deco.kicad_sch (KiCad schematic)
At the start: 12 parts, among them U1 STM32F103C8Tx

Commit message: updated schematic and README
Other:
- note added: "LED Vector"
- note added: "MCU"
- company: Mutronics -> Snailtronics
- moved on the sheet: D1, D10, D2, D3, D4, D5, D6, D7, D8, D9, R1, U1
